Commit message: First semi-successful walking attempt.

File: src/spot_micro/urdf/spot_micro_ai.xacro (robot description, xacro)
@@ -58,5 +58,5 @@
       <axis xyz="1 0 0"/>
       <origin rpy="0 0 0" xyz="${shiftx} ${shifty} 0"/>
-      <limit effort="1000.0" lower="-0.548" upper="0.548" velocity="0.7"/>
+      <limit effort="1000.0" lower="-2.548" upper="2.548" velocity="10.7"/>
       <dynamics damping="0.0" friction="0.5"/>
     </joint>
@@ -117,5 +117,5 @@
       <axis xyz="0 1 0"/>
       <origin rpy="0 0 0" xyz="0 ${shift} 0"/>
-      <limit effort="1000.0" lower="-2.666" upper="1.548" velocity="0.5"/>
+      <limit effort="1000.0" lower="-2.666" upper="1.548" velocity="10.5"/>
       <dynamics damping="0.0" friction="0.0"/>
     </joint>
@@ -160,5 +160,5 @@
       <axis xyz="0 1 0"/>
       <origin rpy="0 0 0" xyz="-0.01 0 -${leg_length}"/>
-      <limit effort="1000.0" lower="-0.1" upper="2.59" velocity="0.5"/>
+      <limit effort="1000.0" lower="-0.1" upper="2.59" velocity="10.5"/>
       <dynamics damping="0.0" friction="0.5"/>
     </joint>
